File: hw/kicad/emacstkl.kicad_pcb (KiCad board)
At the start: 2 copper layers, 348.5 x 129 mm, 227 parts, among them Q1 2N7002, Q2 2N7002, Q3 2N7002, SW1 KEYSW, SW10 KEYSW, SW11 KEYSW, SW12 KEYSW, SW13 KEYSW, SW14 KEYSW, SW15 KEYSW, SW16 KEYSW, SW17 KEYSW, SW18 KEYSW, SW19 KEYSW, SW2 KEYSW, SW20 KEYSW, SW21 KEYSW, SW22 KEYSW, SW23 KEYSW, SW24 KEYSW, SW25 KEYSW, SW26 KEYSW, SW27 KEYSW, SW28 KEYSW, SW3 KEYSW, SW30 KEYSW, SW31 KEYSW, SW32 KEYSW, SW34 KEYSW, SW35 KEYSW, SW36 KEYSW, SW37 KEYSW, SW38 KEYSW, SW39 KEYSW, SW4 KEYSW, SW40 KEYSW, SW41 KEYSW, SW42 KEYSW, SW43 KEYSW, SW44 KEYSW, SW45 KEYSW, SW47 KEYSW, SW48 KEYSW, SW49 KEYSW, SW5 KEYSW, SW51 KEYSW, SW52 KEYSW, SW53 KEYSW, SW54 KEYSW, SW55 KEYSW, SW56 KEYSW, SW57 KEYSW, SW58 KEYSW, SW59 KEYSW, SW6 KEYSW, SW60 KEYSW, SW61 KEYSW, SW62 KEYSW, SW65 KEYSW, SW66 KEYSW, SW67 KEYSW, SW68 KEYSW, SW69 KEYSW, SW7 KEYSW, SW70 KEYSW, SW71 KEYSW, SW72 KEYSW, SW73 KEYSW, SW74 KEYSW, SW76 KEYSW, SW8 KEYSW, SW9 KEYSW, SW92 KEYSW, SW93 KEYSW, SW94 KEYSW, U2 ATmega32A-A, Y2 Crystal

Commit message: ver-2a: Update kicad files
Parts:
- removed C6, C7: 22p, Capacitor_SMD:C_1206_3216Metric_Pad1.33x1.80mm_HandSolder
- removed D95, D96: 3.6V, Diode_SMD:D_MiniMELF_Handsoldering
- removed DL2, DL3: LED, LED_SMD:LED_1206_3216Metric_Pad1.42x1.75mm_HandSolder
- removed Q3: 2N7002, Package_TO_SOT_SMD:SOT-23
- removed R10, R13: 220, Resistor_SMD:R_1206_3216Metric_Pad1.30x1.75mm_HandSolder
- removed R11, R12, R7, R8, R9: 10k, Resistor_SMD:R_1206_3216Metric_Pad1.30x1.75mm_HandSolder
- removed SW-BOOT1: SW_Push, Button_Switch_THT:SW_PUSH_6mm_H4.3mm
- removed Y2: Crystal, Crystal:Crystal_HC49-4H_Vertical
- added C11: 22p, Capacitor_SMD:C_1206_3216Metric_Pad1.33x1.80mm_HandSolder, B.Cu at (162.1, 69.6)
- added C12: 22p, Capacitor_SMD:C_1206_3216Metric_Pad1.33x1.80mm_HandSolder, B.Cu at (163.8, 66.8)
- added C13: 1u, Capacitor_Tantalum_SMD:CP_EIA-3216-18_Kemet-A_HandSolder, B.Cu at (143.8, 54.3)
- added C14: 0.1u, Capacitor_Tantalum_SMD:CP_EIA-3216-18_Kemet-A_HandSolder, B.Cu at (125.7, 63.4)
- added C15: 1u, Capacitor_Tantalum_SMD:CP_EIA-3216-18_Kemet-A_HandSolder, B.Cu at (140.0, 54.3)
- added C16: 0.1u, Capacitor_Tantalum_SMD:CP_EIA-3216-18_Kemet-A_HandSolder, B.Cu at (57.7, 61.4)
- added C17: 0.1u, Capacitor_Tantalum_SMD:CP_EIA-3216-18_Kemet-A_HandSolder, B.Cu at (138.0, 149.6)
- added C18: 1u, Capacitor_Tantalum_SMD:CP_EIA-3216-18_Kemet-A_HandSolder, B.Cu at (138.0, 153.2)
- added C19: 0.1u, Capacitor_Tantalum_SMD:CP_EIA-3216-18_Kemet-A_HandSolder, B.Cu at (145.0, 61.7)
- added DL12: LED, LED_SMD:LED_Kingbright_KPA-3010_3x2x1mm, F.Cu at (24.0, 168.4)
- added DL13: LED, LED_SMD:LED_Kingbright_KPA-3010_3x2x1mm, F.Cu at (42.0, 168.4)
- added DL5: LED, LED_SMD:LED_Kingbright_KPA-3010_3x2x1mm, F.Cu at (163.0, 168.4)
- added DL6: LED, LED_SMD:LED_Kingbright_KPA-3010_3x2x1mm, F.Cu at (60.0, 168.4)
- added DL7: LED, LED_SMD:LED_Kingbright_KPA-3010_3x2x1mm, F.Cu at (73.9, 168.4)
- added DL8: LED, LED_SMD:LED_Kingbright_KPA-3010_3x2x1mm, F.Cu at (105.5, 168.4)
- added DL9: LED, LED_SMD:LED_Kingbright_KPA-3010_3x2x1mm, F.Cu at (128.5, 168.4)
- added H12: MountingHole, MountingHole:MountingHole_4.3mm_M4, F.Cu at (361.0, 69.4)
- added H13: MountingHole, MountingHole:MountingHole_4.3mm_M4, F.Cu at (361.0, 143.4)
- added H14: MountingHole, MountingHole:MountingHole_4.3mm_M4, F.Cu at (24.0, 120.4)
- added J1: Screw_Terminal_01x04, Connector_JST:JST_EH_B4B-EH-A_1x04_P2.50mm_Vertical, B.Cu at (206.8, 163.2)
- added R17: 10k, Resistor_SMD:R_1206_3216Metric_Pad1.30x1.75mm_HandSolder, B.Cu at (147.1, 64.5)
- added R18: 270, Resistor_SMD:R_1206_3216Metric_Pad1.30x1.75mm_HandSolder, B.Cu at (115.1, 159.7)
- added R19: 270, Resistor_SMD:R_1206_3216Metric_Pad1.30x1.75mm_HandSolder, B.Cu at (120.2, 164.8)
- added R20: 270, Resistor_SMD:R_1206_3216Metric_Pad1.30x1.75mm_HandSolder, B.Cu at (128.7, 164.9)
- added R23: 270, Resistor_SMD:R_1206_3216Metric_Pad1.30x1.75mm_HandSolder, B.Cu at (108.2, 153.9)
- added R24: 270, Resistor_SMD:R_1206_3216Metric_Pad1.30x1.75mm_HandSolder, B.Cu at (115.0, 155.9)
- added R25: 10k, Resistor_SMD:R_1206_3216Metric_Pad1.30x1.75mm_HandSolder, B.Cu at (169.6, 150.4)
- added R26: 10k, Resistor_SMD:R_1206_3216Metric_Pad1.30x1.75mm_HandSolder, B.Cu at (178.5, 150.4)
- added R27: 10k, Resistor_SMD:R_1206_3216Metric_Pad1.30x1.75mm_HandSolder, B.Cu at (167.5, 158.9)
- added R28: 10k, Resistor_SMD:R_1206_3216Metric_Pad1.30x1.75mm_HandSolder, B.Cu at (138.0, 156.9)
- added U1: ATmega32U4-A, Package_QFP:TQFP-44_10x10mm_P0.8mm, B.Cu at (137.7, 70.4)
- added U3: PCF8574T, Package_SO:SOIC-16W_7.5x10.3mm_P1.27mm, B.Cu at (126.7, 155.6)
- added Y3: Crystal, Crystal:Crystal_HC49-4H_Vertical, B.Cu at (154.9, 68.5)
- DL1, DL4: footprint LED_SMD:LED_1206_3216Metric_Pad1.42x1.75mm_HandSolder -> LED_SMD:LED_Kingbright_KPA-3010_3x2x1mm
- F1: footprint Fuse:Fuse_0805_2012Metric_Pad1.15x1.40mm_HandSolder -> Resistor_SMD:R_1206_3216Metric_Pad1.30x1.75mm_HandSolder
- H1: footprint MountingHole:MountingHole_3mm_Pad -> MountingHole:MountingHole_4mm_Pad
- H10, H8, H9: footprint MountingHole:MountingHole_3mm -> MountingHole:MountingHole_4mm
- H11, H5: footprint MountingHole:MountingHole_5mm -> MountingHole:MountingHole_6mm
- H2: footprint MountingHole:MountingHole_4mm -> MountingHole:MountingHole_5mm
- R14, R15: value 10k -> 270
- R16: value 220 -> 270
- R3, R4: value 75R -> 22
- R5: value 1.5k -> 1k
- R6: value R -> 0
- RSH1: value 1k -> 1M
- SWBKSP1: footprint fp-Library:SW_CN_Cherry_MX_PCB_2.00u -> fp-Library:SW_CN_S_Cherry_MX_2.00u_PCB
- SWENTER1, SWLSH1: footprint fp-Library:SW_CN_Cherry_MX_PCB_2.25u -> fp-Library:SW_CN_S_Cherry_MX_2.25u_PCB
- SWRSH1: footprint fp-Library:SW_CN_Cherry_MX_PCB_2.75u -> fp-Library:SW_CN_S_Cherry_MX_2.75u_PCB
- SWSPC1: footprint fp-Library:SW_CN_Cherry_MX_PCB_6.25u -> fp-Library:SW_CN_S_Cherry_MX_6.25u_PCB
- U2: value ATmega32A-A -> USBLC6-2SC6; footprint Package_QFP:TQFP-44_10x10mm_P0.8mm -> Package_TO_SOT_SMD:SOT-23-6
- moved DL1 301.3 mm to (19.5, 163.9), turned to 90 degrees
- moved R16 230.1 mm to (108.3, 157.7), turned to 0 degrees
- moved DL4 219.7 mm to (142.5, 168.4)
- moved RL1 203.0 mm to (108.2, 149.6), turned to 180 degrees
- moved AVRISP1 193.1 mm to (349.0, 71.4), turned to 90 degrees
- moved R15 192.3 mm to (167.5, 154.9), turned to 180 degrees
- moved R14 188.0 mm to (167.5, 163.9), turned to 180 degrees
- moved Q2 164.0 mm to (175.0, 154.9), turned to 180 degrees
- moved Q1 153.7 mm to (175.5, 163.9), turned to 180 degrees
- moved SW-RESET1 150.8 mm to (330.8, 67.8)
- moved U2 119.4 mm to (55.1, 53.1)
- moved C9 98.5 mm to (155.2, 63.2)
- moved C8 90.0 mm to (147.6, 76.4)
- moved C5 87.9 mm to (127.3, 75.4)
- moved C3 83.3 mm to (103.0, 68.5)
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Connections:
- DL4 pad 2: Net-(DL4-A) -> +5V
- F1 pad 2: VCC -> Net-(U2-VBUS)
- Q1 pad 3: Net-(DL2-K) -> Net-(Q1-D)
- Q2 pad 3: Net-(DL3-K) -> Net-(Q2-D)
- R14 pad 1: GND -> Net-(Q1-D)
- R14 pad 2: MOSI -> Net-(DL4-K)
- R15 pad 1: MOSI -> Net-(Q2-D)
- R16 pad 1: Net-(DL4-A) -> Net-(DL6-A)
- R16 pad 2: +5V -> Net-(U3-P5)
- R3 pad 1: D- -> DPRO+
- R3 pad 2: DRAW- -> DI+
- R4 pad 1: D+ -> DPRO-
- R4 pad 2: DRAW+ -> DI-
- R5 pad 1: +5V -> GND
- R5 pad 2: DRAW- -> Net-(U1-~{HWB}/PE2)
- SW10 pad 1: col11 -> col10
- SW11 pad 1: col12 -> col11
- SW12 pad 1: col13 -> col12
- SW13 pad 1: col14 -> col13
- SW14 pad 1: col15 -> col14
- SW15 pad 1: col16 -> col15
- SW23 pad 1: col7 -> SCK
- SW24 pad 1: col8 -> MOSI
- SW25 pad 1: col9 -> MISO
- SW30 pad 1: col15 -> col14
- SW31 pad 1: col16 -> col15
- SW32 pad 1: col17 -> col16
- SW40 pad 1: col7 -> SCK
- SW41 pad 1: col8 -> MOSI
- SW42 pad 1: col9 -> MISO
- SW47 pad 1: col15 -> col14
- SW48 pad 1: col16 -> col15
- SW49 pad 1: col17 -> col16
- SW51 pad 1: col17 -> col16
- SW58 pad 1: col7 -> SCK
- SW59 pad 1: col8 -> MOSI
- SW60 pad 1: col9 -> MISO
- SW7 pad 1: col7 -> SCK
- SW71 pad 1: col7 -> SCK
- SW72 pad 1: col8 -> MOSI
- SW73 pad 1: col9 -> MISO
- SW76 pad 1: col16 -> col15
- SW8 pad 1: col8 -> MOSI
- SW9 pad 1: col9 -> MISO
- SW92 pad 1: col15 -> col14
- SW93 pad 1: col16 -> col15
- SW94 pad 1: col17 -> col16
- SWBKSP1 pad 1: col13 -> Net-(DBKSP1-A)
- SWBKSP1 pad 2: Net-(DBKSP1-A) -> col13
- SWENTER1 pad 1: col13 -> Net-(DENTER1-A)
- SWENTER1 pad 2: Net-(DENTER1-A) -> col13
- SWLSH1 pad 1: col0 -> Net-(DLSH1-A)
- SWLSH1 pad 2: Net-(DLSH1-A) -> col0
- SWRALT1 pad 1: col9 -> MISO
- SWRCTL1 pad 1: col14 -> col13
- SWRSH1 pad 1: col13 -> Net-(DRSH1-A)
- SWRSH1 pad 2: Net-(DRSH1-A) -> col13
- SWSPC1 pad 1: col6 -> Net-(DSPC1-A)
- SWSPC1 pad 2: Net-(DSPC1-A) -> col6
- U2 pad 1: MOSI -> D-
- U2 pad 2: MISO -> GND
- U2 pad 3: SCK -> D+
- U2 pad 4: reset-btn -> DPRO+
- U2 pad 5: +5V -> Net-(U2-VBUS)
- U2 pad 6: GND -> DPRO-
- USB1 pad A4: VCC -> Net-(U2-VBUS)
- USB1 pad A6: DRAW+ -> D+
- USB1 pad A7: DRAW- -> D-
- USB1 pad A9: VCC -> Net-(U2-VBUS)
- USB1 pad B4: VCC -> Net-(U2-VBUS)
- USB1 pad B6: DRAW+ -> D+
- USB1 pad B7: DRAW- -> D-
- USB1 pad B9: VCC -> Net-(U2-VBUS)
Routing:
- net col17: track 395.2 -> 0.00 mm, vias 3 -> 0
- net col9: track 261.3 -> 0.00 mm, vias 3 -> 0
- net MISO: track 80.3 -> 341.5 mm, vias 0 -> 3
- net led0: track 259.5 -> 0.00 mm, vias 2 -> 0
- net led1: track 237.3 -> 0.00 mm, vias 2 -> 0
- net SCK: track 90.4 -> 314.0 mm, vias 3 -> 5
- net col8: track 203.9 -> 0.00 mm, vias 3 -> 0
- net col7: track 201.6 -> 0.00 mm, vias 3 -> 0
- net SCL: track 0.00 -> 189.4 mm, vias 0 -> 2
- net SDA: track 0.00 -> 188.5 mm, vias 0 -> 3
- net +5V: track 475.2 -> 579.8 mm, vias 11 -> 4
- net boot: track 101.6 -> 0.00 mm, vias 3 -> 0
- net Net-(DL12-A): track 0.00 -> 99.8 mm, vias 0 -> 1
- net Net-(DL1-A): track 5.46 -> 95.9 mm
- net D-: track 98.9 -> 11.0 mm, vias 2 -> 0
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Other:
- outline, holes or cut-outs redrawn
- board text added: "${PROJECTNAME}^{ver 2.a}"
- board text added: "+5V"
- board text added: "GND"
- board text added: "SCL"
- board text added: "SDA"
- board text removed: "${PROJECTNAME}^{ver 1.a}"
