File: hw/kicad/emacstkl.kicad_sch (KiCad schematic)
At the start: 227 parts, among them Q1 2N7002, Q2 2N7002, Q3 2N7002, SW1 KEYSW, SW10 KEYSW, SW11 KEYSW, SW12 KEYSW, SW13 KEYSW, SW14 KEYSW, SW15 KEYSW, SW16 KEYSW, SW17 KEYSW, SW18 KEYSW, SW19 KEYSW, SW2 KEYSW, SW20 KEYSW, SW21 KEYSW, SW22 KEYSW, SW23 KEYSW, SW24 KEYSW, SW25 KEYSW, SW26 KEYSW, SW27 KEYSW, SW28 KEYSW, SW3 KEYSW, SW30 KEYSW, SW31 KEYSW, SW32 KEYSW, SW34 KEYSW, SW35 KEYSW, SW36 KEYSW, SW37 KEYSW, SW38 KEYSW, SW39 KEYSW, SW4 KEYSW, SW40 KEYSW, SW41 KEYSW, SW42 KEYSW, SW43 KEYSW, SW44 KEYSW, SW45 KEYSW, SW47 KEYSW, SW48 KEYSW, SW49 KEYSW, SW5 KEYSW, SW51 KEYSW, SW52 KEYSW, SW53 KEYSW, SW54 KEYSW, SW55 KEYSW, SW56 KEYSW, SW57 KEYSW, SW58 KEYSW, SW59 KEYSW, SW6 KEYSW, SW60 KEYSW, SW61 KEYSW, SW62 KEYSW, SW65 KEYSW, SW66 KEYSW, SW67 KEYSW, SW68 KEYSW, SW69 KEYSW, SW7 KEYSW, SW70 KEYSW, SW71 KEYSW, SW72 KEYSW, SW73 KEYSW, SW74 KEYSW, SW76 KEYSW, SW8 KEYSW, SW9 KEYSW, SW92 KEYSW, SW93 KEYSW, SW94 KEYSW, U2 ATmega32A-A, Y2 Crystal

Commit message: ver-2a: Update kicad files
Parts:
- removed C6, C7: 22p, Capacitor_SMD:C_1206_3216Metric_Pad1.33x1.80mm_HandSolder, symbol Device:C_Small
- removed D95, D96: 3.6V, Diode_SMD:D_MiniMELF_Handsoldering, symbol Device:D_Zener_Small
- removed DL2, DL3: LED, LED_SMD:LED_1206_3216Metric_Pad1.42x1.75mm_HandSolder, symbol Device:LED
- removed Q3: 2N7002, Package_TO_SOT_SMD:SOT-23, symbol Transistor_FET:2N7002
- removed R10, R13: 220, Resistor_SMD:R_1206_3216Metric_Pad1.30x1.75mm_HandSolder, symbol Device:R_Small
- removed R11, R12, R7, R8, R9: 10k, Resistor_SMD:R_1206_3216Metric_Pad1.30x1.75mm_HandSolder, symbol Device:R_Small
- removed SW-BOOT1: SW_Push, Button_Switch_THT:SW_PUSH_6mm_H4.3mm, symbol Switch:SW_Push
- removed U2: ATmega32A-A, Package_QFP:TQFP-44_10x10mm_P0.8mm, symbol MCU_Microchip_ATmega:ATmega32A-A
- removed Y2: Crystal, Crystal:Crystal_HC49-4H_Vertical, symbol Device:Crystal
- added C11, C12: 22p, Capacitor_SMD:C_1206_3216Metric_Pad1.33x1.80mm_HandSolder, symbol Device:C_Small
- added C13, C15, C18: 1u, Capacitor_Tantalum_SMD:CP_EIA-3216-18_Kemet-A_HandSolder, symbol Device:C_Small
- added C14, C16, C17, C19: 0.1u, Capacitor_Tantalum_SMD:CP_EIA-3216-18_Kemet-A_HandSolder, symbol Device:C_Small
- added DL12, DL13, DL5, DL6, DL7, DL8, DL9: LED, LED_SMD:LED_Kingbright_KPA-3010_3x2x1mm, symbol Device:LED
- added H12, H13, H14: MountingHole, MountingHole:MountingHole_4.3mm_M4, symbol Mechanical:MountingHole
- added J1: Screw_Terminal_01x04, Connector_JST:JST_EH_B4B-EH-A_1x04_P2.50mm_Vertical, symbol Connector:Screw_Terminal_01x04
- added R17, R25, R26, R27, R28: 10k, Resistor_SMD:R_1206_3216Metric_Pad1.30x1.75mm_HandSolder, symbol Device:R_Small
- added R18, R19, R20, R23, R24: 270, Resistor_SMD:R_1206_3216Metric_Pad1.30x1.75mm_HandSolder, symbol Device:R_Small
- added U1: ATmega32U4-A, Package_QFP:TQFP-44_10x10mm_P0.8mm, symbol MCU_Microchip_ATmega:ATmega32U4-A
- added U2: USBLC6-2SC6, Package_TO_SOT_SMD:SOT-23-6, symbol Power_Protection:USBLC6-2SC6
- added U3: PCF8574T, Package_SO:SOIC-16W_7.5x10.3mm_P1.27mm, symbol Interface_Expansion:PCF8574T
- added Y3: Crystal, Crystal:Crystal_HC49-4H_Vertical, symbol Device:Crystal
- DL1, DL4: footprint LED_SMD:LED_1206_3216Metric_Pad1.42x1.75mm_HandSolder -> LED_SMD:LED_Kingbright_KPA-3010_3x2x1mm
- F1: footprint Fuse:Fuse_0805_2012Metric_Pad1.15x1.40mm_HandSolder -> Resistor_SMD:R_1206_3216Metric_Pad1.30x1.75mm_HandSolder
- H1: footprint MountingHole:MountingHole_3mm_Pad -> MountingHole:MountingHole_4mm_Pad
- H10, H8, H9: footprint MountingHole:MountingHole_3mm -> MountingHole:MountingHole_4mm
- H11, H5: footprint MountingHole:MountingHole_5mm -> MountingHole:MountingHole_6mm
- H2: footprint MountingHole:MountingHole_4mm -> MountingHole:MountingHole_5mm
- R14, R15: value 10k -> 270
- R16: value 220 -> 270
- R3, R4: value 75R -> 22
- R5: value 1.5k -> 1k
- RSH1: value 1k -> 1M
- SWBKSP1: footprint fp-Library:SW_CN_Cherry_MX_PCB_2.00u -> fp-Library:SW_CN_S_Cherry_MX_2.00u_PCB
- SWENTER1, SWLSH1: footprint fp-Library:SW_CN_Cherry_MX_PCB_2.25u -> fp-Library:SW_CN_S_Cherry_MX_2.25u_PCB
- SWRSH1: footprint fp-Library:SW_CN_Cherry_MX_PCB_2.75u -> fp-Library:SW_CN_S_Cherry_MX_2.75u_PCB
- SWSPC1: footprint fp-Library:SW_CN_Cherry_MX_PCB_6.25u -> fp-Library:SW_CN_S_Cherry_MX_6.25u_PCB
Connections:
- net col17 is gone; now on net col16: SW32.1, SW49.1, SW51.1, SW94.1
- net col7 is gone; now on net SCK: SW23.1, SW40.1, SW58.1, SW7.1, SW71.1
- net col8 is gone; now on net MOSI: SW24.1, SW41.1, SW59.1, SW72.1, SW8.1
- net col9 is gone; now on net MISO: SW25.1, SW42.1, SW60.1, SW73.1, SW9.1, SWRALT1.1
- net +5V: now also DL4.2 (A), C13.1, C17.1, C18.1, DL5.2 (A), J1.2 (Pin_2), R17.1, R25.1, R26.1, U1.14 (VCC), U1.2 (UVCC), U1.24 (AVCC), U1.34 (VCC), U1.44 (AVCC), U1.7 (VBUS), U3.16 (VDD); no longer R16.2, R5.1
- net D+: now also USB1.A6 (DP1), USB1.B6 (DP2), U2.3 (I/O2); no longer R4.1
- net D-: now also USB1.A7 (DN1), USB1.B7 (DN2), U2.1 (I/O1); no longer R3.1
- net GND: now also R5.1, C11.2, C12.2, C13.2, C14.2, C15.2, C16.2, C17.2, C18.2, C19.2, DL12.1 (K), DL13.1 (K), DL6.1 (K), DL7.1 (K), DL8.1 (K), DL9.1 (K), J1.1 (Pin_1), U1.15 (GND), U1.23 (GND), U1.35 (GND), U1.43 (GND), U1.5 (UGND), U2.2 (GND), U3.1 (A0), U3.2 (A1), U3.3 (A2), U3.8 (GND); no longer R14.1
- net MISO: now also U1.11 (PB3)
- net MOSI: now also U1.10 (PB2); no longer R14.2, R15.1
- net SCK: now also U1.9 (PB1)
- net col0: now also SWLSH1.2, U1.1 (PE6); no longer SWLSH1.1
- net col1: now also U1.41 (PF0)
- net col10: now also SW10.1, U1.12 (PB7)
- net col11: now also SW11.1, U1.27 (PD7); no longer SW10.1
- net col12: now also SW12.1, U1.28 (PB4); no longer SW11.1
- net col13: now also SW13.1, SWBKSP1.2, SWENTER1.2, SWRCTL1.1, SWRSH1.2, U1.20 (PD2); no longer SW12.1, SWBKSP1.1, SWENTER1.1, SWRSH1.1
- net col14: now also SW14.1, SW30.1, SW47.1, SW92.1, U1.21 (PD3); no longer SW13.1, SWRCTL1.1
- net col15: now also SW15.1, SW31.1, SW48.1, SW76.1, SW93.1, U1.22 (PD5); no longer SW14.1, SW30.1, SW47.1, SW92.1
- net col16: now also U1.25 (PD4); no longer SW15.1, SW31.1, SW48.1, SW76.1, SW93.1
- net col2: now also U1.40 (PF1)
- net col3: now also U1.39 (PF4)
- net col4: now also U1.38 (PF5)
- net col5: now also U1.37 (PF6)
- net col6: now also SWSPC1.2, U1.26 (PD6); no longer SWSPC1.1
- net reset-btn: now also C19.1, R17.2, U1.13 (~{RESET})
- net row0: now also U1.8 (PB0)
- net row1: now also U1.36 (PF7)
- net row2: now also U1.29 (PB5)
- net row3: now also U1.30 (PB6)
- net row4: now also U1.31 (PC6)
- net row5: now also U1.32 (PC7)
- net at DLSH1.2 (A): now also SWLSH1.1; no longer SWLSH1.2
- net at R15.2: now also DL5.1 (K)
- net at DL4.1 (K): now also R14.2
- net at R16.1: now also DL6.2 (A); no longer DL4.2 (A)
- net at DSPC1.2 (A): now also SWSPC1.1; no longer SWSPC1.2
- net at Q1.3 (D): now also R14.1
- net at Q1.1 (G): now also R27.2
- net at Q2.1 (G): now also R28.2
- net at Q2.3 (D): now also R15.1
- net at DBKSP1.2 (A): now also SWBKSP1.1; no longer SWBKSP1.2
- net at DRSH1.2 (A): now also SWRSH1.1; no longer SWRSH1.2
- net at DENTER1.2 (A): now also SWENTER1.1; no longer SWENTER1.2
- removed net DRAW+: R4.2, USB1.A6 (DP1), USB1.B6 (DP2)
- removed net DRAW-: R3.2, R5.2, USB1.A7 (DN1), USB1.B7 (DN2)
- net VCC: no longer names the net of F1.2, USB1.A4 (VBUS), USB1.A9 (VBUS), USB1.B4 (VBUS), USB1.B9 (VBUS)
- net VCC: now also C16.1, U2.5 (VBUS)
- new net: C15.1, U1.6 (UCAP)
- new net: DL9.2 (A), R20.1
- new net: DL12.2 (A), R23.1
- new net: R27.1, U3.5 (P1)
- new net: R28.1, U3.4 (P0)
- new net: R20.2, U3.6 (P2)
- new net: DL8.2 (A), R19.1
- new net: R19.2, U3.7 (P3)
- new net: R16.2, U3.10 (P5)
- new net: R24.2, U3.11 (P6)
- new net: R23.2, U3.12 (P7)
- new net: R18.2, U3.9 (P4)
- new net: C11.1, U1.17 (XTAL1), Y3.1
- new net: C12.1, U1.16 (XTAL2), Y3.2
- new net: DL13.2 (A), R24.1
- new net: C14.1, U1.42 (AREF)
- new net: DL7.2 (A), R18.1
- new net: R5.2, U1.33 (~{HWB}/PE2)
- new net DI+: R3.2, U1.4 (D+)
- new net DI-: R4.2, U1.3 (D-)
- new net DPRO+: R3.1, U2.4 (I/O2)
- new net DPRO-: R4.1, U2.6 (I/O1)
- new net SCL: J1.4 (Pin_4), R25.2, U1.18 (PD0), U3.14 (SCL)
- new net SDA: J1.3 (Pin_3), R26.2, U1.19 (PD1), U3.15 (SDA)
- no-connect marks 3 -> 2
Other:
- note added: "add tvs diodes"
- moved on the sheet: AVRISP1, D10, D11, D12, D13, DL1, DRCTL1, F1, H10, H11, H2, H3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
